File: Circuit.sch (EAGLE design)
At the start: 120 parts, among them IC1 LM1117T-3.3-V

Commit message: Removed pointless resistors
Parts:
- removed R12, R13, R20, R21, R36, R37: 2.2K, resistor:R-EU_R0603
Connections:
- net +3V3: no longer R12.1, R13.1, R20.1, R21.1, R36.1, R37.1
- net B1_SC1: no longer R13.2
- net B1_SC2: no longer R20.2
- net B1_SD1: no longer R12.2
- net B1_SD2: no longer R21.2
- net B2_SC2: no longer R36.2
- net B2_SD2: no longer R37.2
Changed lines of the file:
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@@
 <part name="C29" library="SparkFun" deviceset="CAP" device="0603-CAP" value="10uF"/>
 <part name="GND27" library="supply1" deviceset="GND" device=""/>
-<part name="R20" library="resistor" deviceset="R-EU_" device="R0603" value="2.2K"/>
-<part name="R21" library="resistor" deviceset="R-EU_" device="R0603" value="2.2K"/>
 <part name="+3V35" library="supply1" deviceset="+3V3" device=""/>
 <part name="C30" library="SparkFun" deviceset="CAP" device="0603-CAP" value="10nF"/>
@@
 <part name="C56" library="SparkFun" deviceset="CAP" device="0603-CAP" value="10uF"/>
 <part name="GND29" library="supply1" deviceset="GND" device=""/>
-<part name="R36" library="resistor" deviceset="R-EU_" device="R0603" value="2.2K"/>
-<part name="R37" library="resistor" deviceset="R-EU_" device="R0603" value="2.2K"/>
 <part name="+3V39" library="supply1" deviceset="+3V3" device=""/>
 <part name="C57" library="SparkFun" deviceset="CAP" device="0603-CAP" value="10nF"/>
@@
 <part name="R28" library="resistor" deviceset="R-EU_" device="R0603" value="2.2K"/>
 <part name="+3V49" library="supply1" deviceset="+3V3" device=""/>
-<part name="R12" library="resistor" deviceset="R-EU_" device="R0603" value="2.2K"/>
-<part name="R13" library="resistor" deviceset="R-EU_" device="R0603" value="2.2K"/>
-<part name="+3V50" library="supply1" deviceset="+3V3" device=""/>
 <part name="R27" library="resistor" deviceset="R-EU_" device="R0603" value="2.2K"/>
 <part name="R29" library="resistor" deviceset="R-EU_" device="R0603" value="2.2K"/>
@@
 <instance part="C29" gate="G$1" x="27.94" y="27.94"/>
 <instance part="GND27" gate="1" x="38.1" y="-2.54"/>
-<instance part="R20" gate="G$1" x="83.82" y="53.34" rot="R180"/>
-<instance part="R21" gate="G$1" x="91.44" y="48.26" rot="R180"/>
 <instance part="+3V35" gate="G$1" x="99.06" y="60.96"/>
 <instance part="C30" gate="G$1" x="81.28" y="17.78"/>
@@
 <instance part="C56" gate="G$1" x="256.54" y="27.94"/>
 <instance part="GND29" gate="1" x="266.7" y="-2.54"/>
-<instance part="R36" gate="G$1" x="312.42" y="53.34" rot="R180"/>
-<instance part="R37" gate="G$1" x="320.04" y="48.26" rot="R180"/>
 <instance part="+3V39" gate="G$1" x="327.66" y="60.96"/>
 <instance part="C57" gate="G$1" x="309.88" y="17.78"/>
@@
 <instance part="R28" gate="G$1" x="215.9" y="345.44" rot="R180"/>
 <instance part="+3V49" gate="G$1" x="233.68" y="350.52" rot="R270"/>
-<instance part="R12" gate="G$1" x="-17.78" y="160.02" rot="R180"/>
-<instance part="R13" gate="G$1" x="-5.08" y="152.4" rot="R180"/>
-<instance part="+3V50" gate="G$1" x="20.32" y="160.02" rot="R270"/>
 <instance part="R27" gate="G$1" x="208.28" y="160.02" rot="R180"/>
 <instance part="R29" gate="G$1" x="220.98" y="152.4" rot="R180"/>
@@
 </segment>
 <segment>
-<pinref part="R20" gate="G$1" pin="1"/>
-<wire x1="88.9" y1="53.34" x2="99.06" y2="53.34" width="0.1524" layer="91"/>
-<pinref part="R21" gate="G$1" pin="1"/>
-<wire x1="99.06" y1="53.34" x2="99.06" y2="48.26" width="0.1524" layer="91"/>
-<wire x1="99.06" y1="48.26" x2="96.52" y2="48.26" width="0.1524" layer="91"/>
-<wire x1="99.06" y1="53.34" x2="99.06" y2="58.42" width="0.1524" layer="91"/>
 <pinref part="+3V35" gate="G$1" pin="+3V3"/>
 <pinref part="L3G_2" gate="G$1" pin="CS"/>
 <wire x1="73.66" y1="30.48" x2="99.06" y2="30.48" width="0.1524" layer="91"/>
 <wire x1="99.06" y1="30.48" x2="99.06" y2="33.02" width="0.1524" layer="91"/>
-<junction x="99.06" y="53.34"/>
-<junction x="99.06" y="48.26"/>
 <pinref part="L3G_2" gate="G$1" pin="SDO"/>
-<wire x1="99.06" y1="33.02" x2="99.06" y2="48.26" width="0.1524" layer="91"/>
+<wire x1="99.06" y1="33.02" x2="99.06" y2="58.42" width="0.1524" layer="91"/>
 <wire x1="73.66" y1="33.02" x2="99.06" y2="33.02" width="0.1524" layer="91"/>
 <junction x="99.06" y="33.02"/>
@@
 </segment>
 <segment>
-<pinref part="R36" gate="G$1" pin="1"/>
-<wire x1="317.5" y1="53.34" x2="327.66" y2="53.34" width="0.1524" layer="91"/>
-<pinref part="R37" gate="G$1" pin="1"/>
-<wire x1="327.66" y1="53.34" x2="327.66" y2="48.26" width="0.1524" layer="91"/>
-<wire x1="327.66" y1="48.26" x2="325.12" y2="48.26" width="0.1524" layer="91"/>
-<wire x1="327.66" y1="53.34" x2="327.66" y2="58.42" width="0.1524" layer="91"/>
 <pinref part="+3V39" gate="G$1" pin="+3V3"/>
 <pinref part="L3G_4" gate="G$1" pin="CS"/>
 <wire x1="302.26" y1="30.48" x2="327.66" y2="30.48" width="0.1524" layer="91"/>
 <wire x1="327.66" y1="30.48" x2="327.66" y2="33.02" width="0.1524" layer="91"/>
-<junction x="327.66" y="53.34"/>
-<junction x="327.66" y="48.26"/>
 <pinref part="L3G_4" gate="G$1" pin="SDO"/>
-<wire x1="327.66" y1="33.02" x2="327.66" y2="48.26" width="0.1524" layer="91"/>
+<wire x1="327.66" y1="33.02" x2="327.66" y2="58.42" width="0.1524" layer="91"/>
 <wire x1="302.26" y1="33.02" x2="327.66" y2="33.02" width="0.1524" layer="91"/>
 <junction x="327.66" y="33.02"/>
@@
 </segment>
 <segment>
-<pinref part="R12" gate="G$1" pin="1"/>
-<wire x1="-12.7" y1="160.02" x2="7.62" y2="160.02" width="0.1524" layer="91"/>
-<wire x1="7.62" y1="160.02" x2="7.62" y2="152.4" width="0.1524" layer="91"/>
-<pinref part="R13" gate="G$1" pin="1"/>
-<wire x1="7.62" y1="152.4" x2="0" y2="152.4" width="0.1524" layer="91"/>
-<wire x1="7.62" y1="160.02" x2="17.78" y2="160.02" width="0.1524" layer="91"/>
-<pinref part="+3V50" gate="G$1" pin="+3V3"/>
-<junction x="7.62" y="160.02"/>
-</segment>
-<segment>
 <pinref part="R27" gate="G$1" pin="1"/>
 <wire x1="213.36" y1="160.02" x2="233.68" y2="160.02" width="0.1524" layer="91"/>
@@
 <segment>
 <pinref part="ITG3" gate="G$1" pin="SDA"/>
-<wire x1="-33.02" y1="144.78" x2="-30.48" y2="144.78" width="0.1524" layer="91"/>
 <label x="-12.7" y="147.32" size="1.778" layer="95" rot="R180"/>
-<pinref part="R12" gate="G$1" pin="2"/>
-<wire x1="-30.48" y1="144.78" x2="-12.7" y2="144.78" width="0.1524" layer="91"/>
-<wire x1="-22.86" y1="160.02" x2="-30.48" y2="160.02" width="0.1524" layer="91"/>
-<wire x1="-30.48" y1="160.02" x2="-30.48" y2="144.78" width="0.1524" layer="91"/>
-<junction x="-30.48" y="144.78"/>
+<wire x1="-33.02" y1="144.78" x2="-12.7" y2="144.78" width="0.1524" layer="91"/>
 </segment>
 <segment>
@@
 <segment>
 <pinref part="ITG3" gate="G$1" pin="SCL"/>
-<wire x1="-33.02" y1="139.7" x2="-25.4" y2="139.7" width="0.1524" layer="91"/>
 <label x="-12.7" y="142.24" size="1.778" layer="95" rot="R180"/>
-<wire x1="-25.4" y1="139.7" x2="-12.7" y2="139.7" width="0.1524" layer="91"/>
-<wire x1="-25.4" y1="139.7" x2="-25.4" y2="152.4" width="0.1524" layer="91"/>
-<pinref part="R13" gate="G$1" pin="2"/>
-<wire x1="-25.4" y1="152.4" x2="-10.16" y2="152.4" width="0.1524" layer="91"/>
-<junction x="-25.4" y="139.7"/>
+<wire x1="-33.02" y1="139.7" x2="-12.7" y2="139.7" width="0.1524" layer="91"/>
 </segment>
 <segment>
@@
 </segment>
 <segment>
-<pinref part="R20" gate="G$1" pin="2"/>
-<wire x1="78.74" y1="53.34" x2="76.2" y2="53.34" width="0.1524" layer="91"/>
-<wire x1="76.2" y1="53.34" x2="76.2" y2="38.1" width="0.1524" layer="91"/>
 <pinref part="L3G_2" gate="G$1" pin="SCL"/>
-<wire x1="73.66" y1="38.1" x2="76.2" y2="38.1" width="0.1524" layer="91"/>
 <label x="93.98" y="40.64" size="1.778" layer="95" rot="R180"/>
-<junction x="76.2" y="38.1"/>
-<wire x1="76.2" y1="38.1" x2="93.98" y2="38.1" width="0.1524" layer="91"/>
+<wire x1="73.66" y1="38.1" x2="93.98" y2="38.1" width="0.1524" layer="91"/>
 </segment>
 </net>
@@
 </segment>
 <segment>
-<pinref part="R21" gate="G$1" pin="2"/>
-<wire x1="86.36" y1="48.26" x2="81.28" y2="48.26" width="0.1524" layer="91"/>
-<wire x1="81.28" y1="48.26" x2="81.28" y2="35.56" width="0.1524" layer="91"/>
 <pinref part="L3G_2" gate="G$1" pin="SDA/SDI"/>
-<wire x1="73.66" y1="35.56" x2="81.28" y2="35.56" width="0.1524" layer="91"/>
 <label x="93.98" y="38.1" size="1.778" layer="95" rot="R180"/>
-<junction x="81.28" y="35.56"/>
-<wire x1="81.28" y1="35.56" x2="93.98" y2="35.56" width="0.1524" layer="91"/>
+<wire x1="73.66" y1="35.56" x2="93.98" y2="35.56" width="0.1524" layer="91"/>
 </segment>
 </net>
@@
 </segment>
 <segment>
-<pinref part="R36" gate="G$1" pin="2"/>
-<wire x1="307.34" y1="53.34" x2="304.8" y2="53.34" width="0.1524" layer="91"/>
-<wire x1="304.8" y1="53.34" x2="304.8" y2="38.1" width="0.1524" layer="91"/>
 <pinref part="L3G_4" gate="G$1" pin="SCL"/>
-<wire x1="302.26" y1="38.1" x2="304.8" y2="38.1" width="0.1524" layer="91"/>
-<junction x="304.8" y="38.1"/>
-<wire x1="304.8" y1="38.1" x2="322.58" y2="38.1" width="0.1524" layer="91"/>
+<wire x1="302.26" y1="38.1" x2="322.58" y2="38.1" width="0.1524" layer="91"/>
 <label x="322.58" y="40.64" size="1.778" layer="95" rot="R180"/>
 </segment>
@@
 </segment>
 <segment>
-<pinref part="R37" gate="G$1" pin="2"/>
-<wire x1="314.96" y1="48.26" x2="309.88" y2="48.26" width="0.1524" layer="91"/>
-<wire x1="309.88" y1="48.26" x2="309.88" y2="35.56" width="0.1524" layer="91"/>
 <pinref part="L3G_4" gate="G$1" pin="SDA/SDI"/>
-<wire x1="302.26" y1="35.56" x2="309.88" y2="35.56" width="0.1524" layer="91"/>
-<junction x="309.88" y="35.56"/>
-<wire x1="309.88" y1="35.56" x2="322.58" y2="35.56" width="0.1524" layer="91"/>
+<wire x1="302.26" y1="35.56" x2="322.58" y2="35.56" width="0.1524" layer="91"/>
 <label x="322.58" y="38.1" size="1.778" layer="95" rot="R180"/>
 </segment>

Commit message: About to find a load of problems. Ignorance is bliss.
Connections:
- removed net N$11: R15.1
- removed net N$12: R18.1
- removed net N$18: R31.1
- removed net N$19: R34.1
- net I1_AUXCLK: now also R15.1
- net I1_AUXSDA: now also R18.1
- net I2_AUXCLK: now also R31.1
- net I2_AUXSDA: now also R34.1
Changed lines of the file:
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@@
 <pinref part="ITG2" gate="G$1" pin="VDD"/>
 <wire x1="195.58" y1="215.9" x2="200.66" y2="215.9" width="0.1524" layer="91"/>
+<junction x="200.66" y="215.9"/>
 </segment>
 <segment>
@@
 </segment>
 </net>
-<net name="N$11" class="0">
-<segment>
-<pinref part="R15" gate="G$1" pin="1"/>
-<wire x1="71.12" y1="233.68" x2="71.12" y2="228.6" width="0.1524" layer="91"/>
-</segment>
-</net>
-<net name="N$12" class="0">
-<segment>
-<pinref part="R18" gate="G$1" pin="1"/>
-<wire x1="78.74" y1="233.68" x2="78.74" y2="226.06" width="0.1524" layer="91"/>
-</segment>
-</net>
 <net name="N$13" class="0">
 <segment>
@@
 </segment>
 </net>
-<net name="N$18" class="0">
-<segment>
-<pinref part="R31" gate="G$1" pin="1"/>
-<wire x1="299.72" y1="233.68" x2="299.72" y2="228.6" width="0.1524" layer="91"/>
-</segment>
-</net>
-<net name="N$19" class="0">
-<segment>
-<pinref part="R34" gate="G$1" pin="1"/>
-<wire x1="307.34" y1="233.68" x2="307.34" y2="226.06" width="0.1524" layer="91"/>
-</segment>
-</net>
 <net name="N$20" class="0">
 <segment>
@@
 <segment>
 <pinref part="ACL_3" gate="G$1" pin="SDA"/>
-<wire x1="66.04" y1="226.06" x2="88.9" y2="226.06" width="0.1524" layer="91"/>
+<wire x1="66.04" y1="226.06" x2="78.74" y2="226.06" width="0.1524" layer="91"/>
+<wire x1="78.74" y1="226.06" x2="88.9" y2="226.06" width="0.1524" layer="91"/>
 <wire x1="88.9" y1="226.06" x2="88.9" y2="223.52" width="0.1524" layer="91"/>
 <wire x1="88.9" y1="223.52" x2="104.14" y2="223.52" width="0.1524" layer="91"/>
 <label x="104.14" y="226.06" size="1.778" layer="95" rot="R180"/>
+<pinref part="R18" gate="G$1" pin="1"/>
+<wire x1="78.74" y1="233.68" x2="78.74" y2="226.06" width="0.1524" layer="91"/>
+<junction x="78.74" y="226.06"/>
 </segment>
 </net>
@@
 <segment>
 <pinref part="ACL_3" gate="G$1" pin="SCL"/>
-<wire x1="66.04" y1="228.6" x2="104.14" y2="228.6" width="0.1524" layer="91"/>
+<wire x1="66.04" y1="228.6" x2="71.12" y2="228.6" width="0.1524" layer="91"/>
 <label x="104.14" y="231.14" size="1.778" layer="95" rot="R180"/>
+<pinref part="R15" gate="G$1" pin="1"/>
+<wire x1="71.12" y1="228.6" x2="104.14" y2="228.6" width="0.1524" layer="91"/>
+<wire x1="71.12" y1="233.68" x2="71.12" y2="228.6" width="0.1524" layer="91"/>
+<junction x="71.12" y="228.6"/>
 </segment>
 </net>
@@
 <segment>
 <pinref part="ACL_4" gate="G$1" pin="SDA"/>
-<wire x1="294.64" y1="226.06" x2="320.04" y2="226.06" width="0.1524" layer="91"/>
+<wire x1="294.64" y1="226.06" x2="307.34" y2="226.06" width="0.1524" layer="91"/>
+<wire x1="307.34" y1="226.06" x2="320.04" y2="226.06" width="0.1524" layer="91"/>
 <wire x1="320.04" y1="226.06" x2="320.04" y2="223.52" width="0.1524" layer="91"/>
 <wire x1="320.04" y1="223.52" x2="335.28" y2="223.52" width="0.1524" layer="91"/>
 <label x="335.28" y="226.06" size="1.778" layer="95" rot="R180"/>
+<pinref part="R34" gate="G$1" pin="1"/>
+<wire x1="307.34" y1="233.68" x2="307.34" y2="226.06" width="0.1524" layer="91"/>
+<junction x="307.34" y="226.06"/>
 </segment>
 </net>
@@
 <segment>
 <pinref part="ACL_4" gate="G$1" pin="SCL"/>
-<wire x1="294.64" y1="228.6" x2="335.28" y2="228.6" width="0.1524" layer="91"/>
+<wire x1="294.64" y1="228.6" x2="299.72" y2="228.6" width="0.1524" layer="91"/>
 <label x="335.28" y="231.14" size="1.778" layer="95" rot="R180"/>
-</segment>
-</net>
+<pinref part="R31" gate="G$1" pin="1"/>
+<wire x1="299.72" y1="228.6" x2="335.28" y2="228.6" width="0.1524" layer="91"/>
+<wire x1="299.72" y1="233.68" x2="299.72" y2="228.6" width="0.1524" layer="91"/>
+<junction x="299.72" y="228.6"/>
+</segment>
+</net>

Commit message: Magnometer left
Connections:
- removed net N$22: ITG4.VDD
- removed net N$24: C41.1
- removed net N$25: R16.1
- removed net N$26: R19.1
- net +3V3: now also C41.1, ITG4.VDD
- net I3_AUXCLK: now also R16.1
- net I3_AUXSDA: now also R19.1
Changed lines of the file:
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@@
 <part name="R29" library="resistor" deviceset="R-EU_" device="R0603" value="2.2K"/>
 <part name="+3V51" library="supply1" deviceset="+3V3" device=""/>
+<part name="+3V31" library="supply1" deviceset="+3V3" device=""/>
 </parts>
 <sheets>
@@
 <instance part="R29" gate="G$1" x="220.98" y="152.4" rot="R180"/>
 <instance part="+3V51" gate="G$1" x="246.38" y="160.02" rot="R270"/>
+<instance part="+3V31" gate="G$1" x="208.28" y="119.38" rot="R270"/>
 </instances>
 <busses>
@@
 <pinref part="ITG1" gate="G$1" pin="VDD"/>
 <wire x1="-33.02" y1="215.9" x2="-27.94" y2="215.9" width="0.1524" layer="91"/>
+<junction x="-27.94" y="215.9"/>
 </segment>
 <segment>
@@
 <pinref part="ITG3" gate="G$1" pin="VDD"/>
 <wire x1="-33.02" y1="119.38" x2="-27.94" y2="119.38" width="0.1524" layer="91"/>
+<junction x="-27.94" y="119.38"/>
 </segment>
 <segment>
@@
 <wire x1="226.06" y1="350.52" x2="231.14" y2="350.52" width="0.1524" layer="91"/>
 <pinref part="+3V49" gate="G$1" pin="+3V3"/>
+<junction x="226.06" y="350.52"/>
 </segment>
 <segment>
@@
 <wire x1="233.68" y1="152.4" x2="233.68" y2="160.02" width="0.1524" layer="91"/>
 <junction x="233.68" y="160.02"/>
+</segment>
+<segment>
+<pinref part="ITG4" gate="G$1" pin="VDD"/>
+<wire x1="195.58" y1="119.38" x2="200.66" y2="119.38" width="0.1524" layer="91"/>
+<pinref part="C41" gate="G$1" pin="1"/>
+<wire x1="200.66" y1="119.38" x2="205.74" y2="119.38" width="0.1524" layer="91"/>
+<wire x1="200.66" y1="119.38" x2="200.66" y2="116.84" width="0.1524" layer="91"/>
+<junction x="200.66" y="119.38"/>
+<pinref part="+3V31" gate="G$1" pin="+3V3"/>
 </segment>
 </net>
@@
 </segment>
 </net>
-<net name="N$25" class="0">
-<segment>
-<pinref part="R16" gate="G$1" pin="1"/>
-<wire x1="71.12" y1="137.16" x2="71.12" y2="132.08" width="0.1524" layer="91"/>
-</segment>
-</net>
-<net name="N$26" class="0">
-<segment>
-<pinref part="R19" gate="G$1" pin="1"/>
-<wire x1="78.74" y1="137.16" x2="78.74" y2="129.54" width="0.1524" layer="91"/>
-</segment>
-</net>
 <net name="N$27" class="0">
 <segment>
@@
 <segment>
 <pinref part="ACL_5" gate="G$1" pin="SDA"/>
-<wire x1="66.04" y1="129.54" x2="88.9" y2="129.54" width="0.1524" layer="91"/>
+<wire x1="66.04" y1="129.54" x2="78.74" y2="129.54" width="0.1524" layer="91"/>
+<wire x1="78.74" y1="129.54" x2="88.9" y2="129.54" width="0.1524" layer="91"/>
 <wire x1="88.9" y1="129.54" x2="88.9" y2="127" width="0.1524" layer="91"/>
 <wire x1="88.9" y1="127" x2="104.14" y2="127" width="0.1524" layer="91"/>
 <label x="104.14" y="129.54" size="1.778" layer="95" rot="R180"/>
+<pinref part="R19" gate="G$1" pin="1"/>
+<wire x1="78.74" y1="137.16" x2="78.74" y2="129.54" width="0.1524" layer="91"/>
+<junction x="78.74" y="129.54"/>
 </segment>
 </net>
@@
 <segment>
 <pinref part="ACL_5" gate="G$1" pin="SCL"/>
-<wire x1="66.04" y1="132.08" x2="104.14" y2="132.08" width="0.1524" layer="91"/>
+<wire x1="66.04" y1="132.08" x2="71.12" y2="132.08" width="0.1524" layer="91"/>
 <label x="104.14" y="134.62" size="1.778" layer="95" rot="R180"/>
+<pinref part="R16" gate="G$1" pin="1"/>
+<wire x1="71.12" y1="132.08" x2="104.14" y2="132.08" width="0.1524" layer="91"/>
+<wire x1="71.12" y1="137.16" x2="71.12" y2="132.08" width="0.1524" layer="91"/>
+<junction x="71.12" y="132.08"/>
 </segment>
 </net>
@@
 <pinref part="R23" gate="G$1" pin="2"/>
 <wire x1="190.5" y1="350.52" x2="193.04" y2="350.52" width="0.1524" layer="91"/>
+<junction x="190.5" y="350.52"/>
 </segment>
 <segment>
@@
 <wire x1="198.12" y1="335.28" x2="198.12" y2="345.44" width="0.1524" layer="91"/>
 <wire x1="198.12" y1="345.44" x2="210.82" y2="345.44" width="0.1524" layer="91"/>
+<junction x="198.12" y="345.44"/>
 </segment>
 <segment>
@@
 </segment>
 </net>
-<net name="N$22" class="0">
-<segment>
-<pinref part="ITG4" gate="G$1" pin="VDD"/>
-<wire x1="195.58" y1="119.38" x2="205.74" y2="119.38" width="0.1524" layer="91"/>
-</segment>
-</net>
-<net name="N$24" class="0">
-<segment>
-<pinref part="C41" gate="G$1" pin="1"/>
-<wire x1="200.66" y1="119.38" x2="200.66" y2="116.84" width="0.1524" layer="91"/>
-</segment>
-</net>

Commit message: Fixing a few schematic errors
Connections:
- removed net N$32: R32.1
- removed net N$33: R35.1
- removed net SCL2: R40.1, U$3.GPIO29
- net CLK2: now also R40.1, U$3.GPIO29
- net I4_AUXCLK: now also R32.1
- net I4_AUXSDA: now also R35.1
Changed lines of the file:
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@@
 <pinref part="GND36" gate="1" pin="GND"/>
 <wire x1="-205.74" y1="340.36" x2="-205.74" y2="337.82" width="0.1524" layer="91"/>
+<junction x="-193.04" y="340.36"/>
 </segment>
 <segment>
@@
 <pinref part="GND38" gate="1" pin="GND"/>
 <wire x1="-205.74" y1="243.84" x2="-205.74" y2="241.3" width="0.1524" layer="91"/>
+<junction x="-193.04" y="243.84"/>
 </segment>
 <segment>
@@
 <wire x1="210.82" y1="124.46" x2="210.82" y2="106.68" width="0.1524" layer="91"/>
 <junction x="210.82" y="106.68"/>
+<junction x="215.9" y="106.68"/>
 </segment>
 <segment>
@@
 <junction x="215.9" y="208.28"/>
 <wire x1="200.66" y1="203.2" x2="215.9" y2="203.2" width="0.1524" layer="91"/>
+<junction x="215.9" y="203.2"/>
 </segment>
 <segment>
@@
 <junction x="-12.7" y="208.28"/>
 <wire x1="-27.94" y1="203.2" x2="-12.7" y2="203.2" width="0.1524" layer="91"/>
+<junction x="-12.7" y="203.2"/>
 </segment>
 <segment>
@@
 <junction x="-12.7" y="111.76"/>
 <wire x1="-27.94" y1="106.68" x2="-12.7" y2="106.68" width="0.1524" layer="91"/>
+<junction x="-12.7" y="106.68"/>
 </segment>
 <segment>
@@
 <wire x1="-147.32" y1="238.76" x2="-134.62" y2="238.76" width="0.1524" layer="91"/>
 <label x="-134.62" y="241.3" size="1.778" layer="95" rot="R180"/>
-</segment>
-</net>
-<net name="SCL2" class="0">
-<segment>
-<pinref part="U$3" gate="G$1" pin="GPIO29"/>
-<wire x1="449.58" y1="154.94" x2="462.28" y2="154.94" width="0.1524" layer="91"/>
-<label x="467.36" y="154.94" size="1.778" layer="95"/>
-<pinref part="R40" gate="G$1" pin="1"/>
-<wire x1="462.28" y1="154.94" x2="472.44" y2="154.94" width="0.1524" layer="91"/>
-<wire x1="462.28" y1="154.94" x2="462.28" y2="157.48" width="0.1524" layer="91"/>
-<junction x="462.28" y="154.94"/>
 </segment>
 </net>
@@
 <wire x1="152.4" y1="312.42" x2="142.24" y2="312.42" width="0.1524" layer="91"/>
 <wire x1="142.24" y1="312.42" x2="142.24" y2="317.5" width="0.1524" layer="91"/>
+<junction x="142.24" y="317.5"/>
 </segment>
 <segment>
@@
 <wire x1="-139.7" y1="139.7" x2="-139.7" y2="144.78" width="0.1524" layer="91"/>
 <junction x="-139.7" y="144.78"/>
+<junction x="-147.32" y="144.78"/>
 </segment>
 <segment>
@@
 <wire x1="-139.7" y1="43.18" x2="-139.7" y2="48.26" width="0.1524" layer="91"/>
 <junction x="-139.7" y="48.26"/>
+<junction x="-147.32" y="48.26"/>
 </segment>
 <segment>
@@
 <label x="-134.62" y="236.22" size="1.778" layer="95" rot="R180"/>
 </segment>
+<segment>
+<pinref part="U$3" gate="G$1" pin="GPIO29"/>
+<wire x1="449.58" y1="154.94" x2="462.28" y2="154.94" width="0.1524" layer="91"/>
+<label x="467.36" y="154.94" size="1.778" layer="95"/>
+<pinref part="R40" gate="G$1" pin="1"/>
+<wire x1="462.28" y1="154.94" x2="472.44" y2="154.94" width="0.1524" layer="91"/>
+<wire x1="462.28" y1="154.94" x2="462.28" y2="157.48" width="0.1524" layer="91"/>
+<junction x="462.28" y="154.94"/>
+</segment>
 </net>
 <net name="N$9" class="0">
@@
 <wire x1="127" y1="165.1" x2="127" y2="88.9" width="0.3048" layer="91"/>
 <label x="127" y="167.64" size="3.81" layer="95"/>
-</segment>
-</net>
-<net name="N$32" class="0">
-<segment>
-<pinref part="R32" gate="G$1" pin="1"/>
-<wire x1="299.72" y1="137.16" x2="299.72" y2="132.08" width="0.1524" layer="91"/>
-</segment>
-</net>
-<net name="N$33" class="0">
-<segment>
-<pinref part="R35" gate="G$1" pin="1"/>
-<wire x1="307.34" y1="137.16" x2="307.34" y2="129.54" width="0.1524" layer="91"/>
 </segment>
 </net>
@@
 <segment>
 <pinref part="ACL_6" gate="G$1" pin="SDA"/>
-<wire x1="294.64" y1="129.54" x2="317.5" y2="129.54" width="0.1524" layer="91"/>
+<wire x1="294.64" y1="129.54" x2="307.34" y2="129.54" width="0.1524" layer="91"/>
+<wire x1="307.34" y1="129.54" x2="317.5" y2="129.54" width="0.1524" layer="91"/>
 <wire x1="317.5" y1="129.54" x2="317.5" y2="127" width="0.1524" layer="91"/>
 <wire x1="317.5" y1="127" x2="332.74" y2="127" width="0.1524" layer="91"/>
 <label x="332.74" y="129.54" size="1.778" layer="95" rot="R180"/>
+<pinref part="R35" gate="G$1" pin="1"/>
+<wire x1="307.34" y1="137.16" x2="307.34" y2="129.54" width="0.1524" layer="91"/>
+<junction x="307.34" y="129.54"/>
 </segment>
 </net>
@@
 <segment>
 <pinref part="ACL_6" gate="G$1" pin="SCL"/>
-<wire x1="294.64" y1="132.08" x2="332.74" y2="132.08" width="0.1524" layer="91"/>
+<wire x1="294.64" y1="132.08" x2="299.72" y2="132.08" width="0.1524" layer="91"/>
 <label x="332.74" y="134.62" size="1.778" layer="95" rot="R180"/>
-</segment>
-</net>
+<pinref part="R32" gate="G$1" pin="1"/>
+<wire x1="299.72" y1="132.08" x2="332.74" y2="132.08" width="0.1524" layer="91"/>
+<wire x1="299.72" y1="137.16" x2="299.72" y2="132.08" width="0.1524" layer="91"/>
+<junction x="299.72" y="132.08"/>
+</segment>
+</net>
