File: Circuit.brd (EAGLE design)
At the start: 99 x 72.1 mm, 115 parts, among them IC1 LM1117T-3.3-V, P1 RASPI-P1RASPI_REV2_P1, P5 RASPI_P5

Commit message: Stash
Parts:
- moved C33 7.57 mm to (37.0, 17.4), turned to 270 degrees
- moved MPU2 1.00 mm to (45.4, 27.0)
- moved C22 0.40 mm to (34.6, 17.4)
Routing:
- net +3V3: track 623.3 -> 638.0 mm, vias 0 -> 2
- net N$7: track 5.64 -> 13.0 mm, vias 0 -> 2
- net M2_AUXCLK: track 27.0 -> 28.5 mm
- net B2_SD2: track 94.8 -> 96.1 mm
- net B2_SD0: track 35.9 -> 36.9 mm
- net N$6: track 5.75 -> 6.74 mm
- net B2_SC2: track 86.2 -> 86.9 mm
- net B2_SC1: track 87.2 -> 87.9 mm
- net B2_SD1: track 90.4 -> 91.0 mm

Commit message: Added via
Routing:
- net B2_SC0: track 37.1 -> 40.6 mm, vias 2 -> 3
- net +3V3: track 638.0 -> 641.3 mm
- net N$6: track 6.74 -> 5.09 mm
- net N$7: track 13.0 -> 14.5 mm
Changed lines of the file:
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@@
 <wire x1="47.4862" y1="25.7033" x2="48.2967" y2="25.7033" width="0.254" layer="1"/>
 <wire x1="48.2967" y1="25.7033" x2="49" y2="25" width="0.254" layer="1"/>
-<wire x1="89" y1="39" x2="89" y2="38.85" width="0" layer="19" extent="1-1"/>
-<wire x1="63.725" y1="35" x2="65.5" y2="35.275" width="0" layer="19" extent="1-1"/>
-<wire x1="36.6" y1="39.85" x2="34.3" y2="39.85" width="0" layer="19" extent="1-1"/>
-<wire x1="72.0862" y1="30.7033" x2="69.7425" y2="29.8784" width="0" layer="19" extent="1-1"/>
-<wire x1="74" y1="30" x2="72.0862" y2="30.7033" width="0" layer="19" extent="1-1"/>
-<wire x1="46.8262" y1="11.1933" x2="44.4825" y2="10.3684" width="0" layer="19" extent="1-1"/>
-<wire x1="61.7" y1="14.45" x2="62.5" y2="12" width="0" layer="19" extent="1-1"/>
-<wire x1="53.2379" y1="30.8784" x2="56.0862" y2="31.7033" width="0" layer="19" extent="1-1"/>
-<wire x1="45.1425" y1="24.8784" x2="47.4895" y2="25.7" width="0" layer="19" extent="1-1"/>
-<wire x1="34.6" y1="18.25" x2="30" y2="19.8" width="0" layer="19" extent="1-1"/>
-<wire x1="34.75" y1="18.25" x2="34.6" y2="18.25" width="0" layer="19" extent="1-1"/>
-<wire x1="38.275" y1="23.0822" x2="36.325" y2="23.0822" width="0" layer="19" extent="1-1"/>
 <wire x1="36.325" y1="23.0822" x2="36.325" y2="21.725" width="0.254" layer="1"/>
 <wire x1="36.325" y1="21.725" x2="36.45" y2="21.6" width="0.254" layer="1"/>
@@
 <wire x1="41.3" y1="24.15" x2="42.25" y2="24.15" width="0.254" layer="1"/>
 <wire x1="42.25" y1="24.15" x2="42.8" y2="23.6" width="0.254" layer="1"/>
-<wire x1="42.8" y1="23.6" x2="44.6379" y2="24.8784" width="0" layer="19" extent="1-16"/>
+<wire x1="42.8" y1="23.6" x2="44.55" y2="23.6" width="0.254" layer="1"/>
+<wire x1="44.55" y1="23.6" x2="45.15" y2="24.2" width="0.254" layer="1"/>
+<wire x1="45.15" y1="24.2" x2="45.15" y2="24.8709" width="0.254" layer="1"/>
+<wire x1="45.15" y1="24.8709" x2="45.1425" y2="24.8784" width="0.254" layer="1"/>
+<wire x1="89" y1="39" x2="89" y2="38.85" width="0" layer="19" extent="1-1"/>
+<wire x1="63.725" y1="35" x2="65.5" y2="35.275" width="0" layer="19" extent="1-1"/>
+<wire x1="36.6" y1="39.85" x2="34.3" y2="39.85" width="0" layer="19" extent="1-1"/>
+<wire x1="72.0862" y1="30.7033" x2="69.7425" y2="29.8784" width="0" layer="19" extent="1-1"/>
+<wire x1="74" y1="30" x2="72.0862" y2="30.7033" width="0" layer="19" extent="1-1"/>
+<wire x1="46.8262" y1="11.1933" x2="44.4825" y2="10.3684" width="0" layer="19" extent="1-1"/>
+<wire x1="61.7" y1="14.45" x2="62.5" y2="12" width="0" layer="19" extent="1-1"/>
+<wire x1="53.2379" y1="30.8784" x2="56.0862" y2="31.7033" width="0" layer="19" extent="1-1"/>
+<wire x1="45.15" y1="24.8709" x2="47.4895" y2="25.7" width="0" layer="19" extent="1-1"/>
+<wire x1="38.275" y1="23.0822" x2="36.325" y2="23.0822" width="0" layer="19" extent="1-1"/>
+<wire x1="40.5" y1="18.2" x2="40.4" y2="20.85" width="0" layer="19" extent="1-1"/>
+<wire x1="34.75" y1="18.25" x2="34.6" y2="18.25" width="0" layer="19" extent="1-1"/>
 </signal>
 <signal name="M1_AUXSDA">
@@
 <contactref element="MPU2" pad="20"/>
 <contactref element="C43" pad="1"/>
-<wire x1="49.5" y1="29.35" x2="49.5" y2="30.5" width="0.254" layer="1"/>
-<wire x1="49.5" y1="30.5" x2="48.8" y2="31.2" width="0.254" layer="1"/>
-<wire x1="48.8" y1="31.2" x2="46.4" y2="31.2" width="0.254" layer="1"/>
-<wire x1="46.4" y1="31.2" x2="46.2" y2="31" width="0.254" layer="1"/>
-<wire x1="46.2" y1="31" x2="46.2" y2="30.102" width="0.254" layer="1"/>
-<wire x1="46.2" y1="30.102" x2="46.1796" y2="29.0816" width="0.254" layer="1"/>
+<wire x1="46.1796" y1="29.0816" x2="46.1796" y2="30.1" width="0.254" layer="1"/>
+<wire x1="46.1796" y1="30.1" x2="49.5" y2="30.1" width="0.254" layer="1"/>
+<wire x1="49.5" y1="30.1" x2="49.5" y2="29.35" width="0.254" layer="1"/>
 </signal>
 <signal name="N$7">
 <contactref element="MPU2" pad="10"/>
 <contactref element="C33" pad="1"/>
-<wire x1="45.6775" y1="24.8784" x2="45.6775" y2="23.8775" width="0.254" layer="1"/>
-<wire x1="45.6775" y1="23.8775" x2="45.4" y2="23.6" width="0.254" layer="1"/>
-<via x="45.4" y="23.6" extent="1-16" drill="0.6"/>
-<wire x1="45.4" y1="23.6" x2="44.6" y2="23.6" width="0.254" layer="16"/>
-<wire x1="44.6" y1="23.6" x2="41" y2="20" width="0.254" layer="16"/>
-<wire x1="41" y1="20" x2="39.2" y2="20" width="0.254" layer="16"/>
 <wire x1="36.95" y1="18.25" x2="39.05" y2="18.25" width="0.254" layer="1"/>
 <wire x1="39.05" y1="18.25" x2="39.15" y2="18.35" width="0.254" layer="1"/>
@@
 <wire x1="39.15" y1="18.35" x2="39.15" y2="19.95" width="0.254" layer="16"/>
 <wire x1="39.15" y1="19.95" x2="39.2" y2="20" width="0.254" layer="16"/>
+<wire x1="39.2" y1="20" x2="43" y2="20" width="0.254" layer="16"/>
+<wire x1="43" y1="20" x2="46.5" y2="23.5" width="0.254" layer="16"/>
+<via x="46.5" y="23.5" extent="1-16" drill="0.6"/>
+<wire x1="46.5" y1="23.5" x2="46.3" y2="23.5" width="0.254" layer="1"/>
+<wire x1="46.3" y1="23.5" x2="45.7" y2="24.1" width="0.254" layer="1"/>
+<wire x1="45.7" y1="24.1" x2="45.7" y2="24.8559" width="0.254" layer="1"/>
+<wire x1="45.7" y1="24.8559" x2="45.6775" y2="24.8784" width="0.254" layer="1"/>
 </signal>
 <signal name="M2_AUXCLK">
@@
 <via x="40.9" y="25.6" extent="1-16" drill="0.6"/>
 <wire x1="49.8" y1="32.9" x2="46.9" y2="32.9" width="0.254" layer="16"/>
-<wire x1="46.9" y1="32.9" x2="44" y2="30" width="0.254" layer="16"/>
+<wire x1="46.9" y1="32.9" x2="45" y2="31" width="0.254" layer="16"/>
+<wire x1="45" y1="31" x2="44" y2="30" width="0.254" layer="16"/>
 <wire x1="44" y1="30" x2="44" y2="27" width="0.254" layer="16"/>
 <wire x1="40.3" y1="26.2" x2="40.9" y2="25.6" width="0.254" layer="1"/>
 <wire x1="44" y1="27" x2="42.3" y2="27" width="0.254" layer="16"/>
 <wire x1="42.3" y1="27" x2="40.9" y2="25.6" width="0.254" layer="16"/>
-<wire x1="44" y1="30" x2="44.6379" y2="29.0816" width="0" layer="19" extent="1-16"/>
+<wire x1="44.6379" y1="29.0816" x2="44.6379" y2="29.6379" width="0.254" layer="1"/>
+<wire x1="44.6379" y1="29.6379" x2="46" y2="31" width="0.254" layer="1"/>
+<via x="46" y="31" extent="1-16" drill="0.6"/>
+<wire x1="46" y1="31" x2="45" y2="31" width="0.254" layer="16"/>
 </signal>
 <signal name="B2_SD1">
@@
 <wire x1="35.3" y1="25.6" x2="39.3" y2="25.6" width="0.254" layer="1"/>
 <wire x1="39.3" y1="25.6" x2="39.3" y2="22.2" width="0.254" layer="1"/>
-<wire x1="48.25" y1="23.45" x2="49.3" y2="23.55" width="0.254" layer="1"/>
+<wire x1="48.2" y1="23.55" x2="49.3" y2="23.55" width="0.254" layer="1"/>
 <wire x1="49.3" y1="23.55" x2="52.15" y2="26.9" width="0.254" layer="1"/>
 <wire x1="52.15" y1="26.9" x2="57.3" y2="26.9" width="0.254" layer="1"/>
@@
 <wire x1="80.1" y1="35.9" x2="80.1" y2="36.9" width="0.254" layer="1"/>
 <wire x1="80.1" y1="36.9" x2="79.3" y2="37.7" width="0.254" layer="1"/>
-<wire x1="46.95" y1="22.15" x2="48.25" y2="23.45" width="0.254" layer="1"/>
-<wire x1="46.95" y1="22.15" x2="44.8" y2="22.2" width="0.254" layer="1"/>
+<wire x1="46.9" y1="22.2" x2="48.2" y2="23.55" width="0.254" layer="1"/>
+<wire x1="46.9" y1="22.2" x2="44.8" y2="22.2" width="0.254" layer="1"/>
 <wire x1="44.8" y1="22.2" x2="44" y2="23" width="0.254" layer="1"/>
 <wire x1="44" y1="23" x2="40.1" y2="23" width="0.254" layer="1"/>
@@
 <wire x1="57.7" y1="25.6" x2="52.7" y2="25.6" width="0.254" layer="1"/>
 <wire x1="52.7" y1="25.6" x2="49.7" y2="22.2" width="0.254" layer="1"/>
-<wire x1="49.7" y1="22.2" x2="48.5" y2="22.2" width="0.254" layer="1"/>
+<wire x1="49.7" y1="22.2" x2="48.65" y2="22.2" width="0.254" layer="1"/>
 <wire x1="33" y1="17" x2="33" y2="9.65" width="0.254" layer="1"/>
 <wire x1="33" y1="9.65" x2="31.85" y2="8.5" width="0.254" layer="1"/>
@@
 <wire x1="33" y1="17" x2="31" y2="19" width="0.254" layer="1"/>
 <wire x1="76.2" y1="27" x2="75.2" y2="26.1" width="0.254" layer="1"/>
-<wire x1="46.45" y1="20.05" x2="35.45" y2="20.05" width="0.254" layer="1"/>
+<wire x1="46.6" y1="20.05" x2="35.45" y2="20.05" width="0.254" layer="1"/>
 <wire x1="35.45" y1="20.05" x2="35.45" y2="21.5" width="0.254" layer="1"/>
 <via x="35.45" y="21.5" extent="1-16" drill="0.6"/>
@@
 <via x="33" y="20" extent="1-16" drill="0.6"/>
 <wire x1="33" y1="20" x2="31" y2="20" width="0.254" layer="1"/>
-<wire x1="48.5" y1="22.2" x2="46.45" y2="20.05" width="0.254" layer="1"/>
+<wire x1="48.65" y1="22.2" x2="46.6" y2="20.05" width="0.254" layer="1"/>
 </signal>
 <signal name="I2C_MUX_2">

Commit message: Going home
Parts:
- moved C37 0.85 mm to (55.4, 29.3)
Routing:
- net +3V3: track 641.3 -> 661.3 mm, vias 2 -> 3
- net N$20: track 2.94 -> 1.69 mm
Changed lines of the file:
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@@
 <element name="R31" library="resistor" package="R0603" value="2.2K" x="44.3" y="38.7"/>
 <element name="R34" library="resistor" package="R0603" value="2.2K" x="47.8" y="38.7"/>
-<element name="C37" library="SparkFun" package="0603-CAP" value="0.1uF" x="55.7" y="28.5"/>
+<element name="C37" library="SparkFun" package="0603-CAP" value="0.1uF" x="55.4" y="29.3"/>
 <element name="C44" library="SparkFun" package="0603-CAP" value="2.2nF" x="58" y="35.8" rot="R270"/>
 <element name="C40" library="SparkFun" package="0603-CAP" value="0.1uF" x="55.8" y="39" rot="R270"/>
@@
 <wire x1="54.7796" y1="30.8784" x2="56.0862" y2="34.2567" width="0" layer="19" extent="1-1"/>
 <wire x1="53.7425" y1="30.8784" x2="54.7796" y2="30.8784" width="0" layer="19" extent="1-1"/>
-<wire x1="56.55" y1="28.5" x2="54.7796" y2="30.8784" width="0" layer="19" extent="1-1"/>
+<wire x1="56.25" y1="29.3" x2="54.7796" y2="30.8784" width="0" layer="19" extent="1-1"/>
 <wire x1="33.725" y1="28.9178" x2="31.85" y2="32.1" width="0" layer="19" extent="1-1"/>
 <wire x1="37.625" y1="28.9178" x2="33.725" y2="28.9178" width="0" layer="19" extent="1-1"/>
@@
 <wire x1="49.5" y1="27.65" x2="47.4862" y2="28.2567" width="0" layer="19" extent="1-1"/>
 <wire x1="46.1796" y1="24.8784" x2="47.4862" y2="28.2567" width="0" layer="19" extent="1-1"/>
-<wire x1="56.15" y1="23.4" x2="56.55" y2="28.5" width="0" layer="19" extent="1-1"/>
+<wire x1="56.15" y1="23.4" x2="56.25" y2="29.3" width="0" layer="19" extent="1-1"/>
 <wire x1="53.15" y1="23.4" x2="56.15" y2="23.4" width="0" layer="19" extent="1-1"/>
 <wire x1="53.75" y1="19.8" x2="53.15" y2="23.4" width="0" layer="19" extent="1-1"/>
@@
 <wire x1="51" y1="26.7" x2="49.6" y2="26.7" width="0.254" layer="1"/>
 <wire x1="49.6" y1="26.7" x2="48.6" y2="25.7" width="0.254" layer="1"/>
-<wire x1="48.6" y1="25.7" x2="47.4895" y2="25.7" width="0.254" layer="1"/>
+<wire x1="48.6" y1="25.7" x2="48.3" y2="25.7" width="0.254" layer="1"/>
 <wire x1="47.4895" y1="25.7" x2="47.4862" y2="25.7033" width="0.254" layer="1"/>
 <wire x1="44.6379" y1="24.8784" x2="45.1425" y2="24.8784" width="0.254" layer="1"/>
 <wire x1="47.4862" y1="25.7033" x2="48.2967" y2="25.7033" width="0.254" layer="1"/>
-<wire x1="48.2967" y1="25.7033" x2="49" y2="25" width="0.254" layer="1"/>
+<wire x1="48.2967" y1="25.7033" x2="48.3" y2="25.7" width="0.254" layer="1"/>
 <wire x1="36.325" y1="23.0822" x2="36.325" y2="21.725" width="0.254" layer="1"/>
 <wire x1="36.325" y1="21.725" x2="36.45" y2="21.6" width="0.254" layer="1"/>
 <wire x1="36.45" y1="21.6" x2="36.45" y2="21.15" width="0.254" layer="1"/>
 <wire x1="36.45" y1="21.15" x2="36.75" y2="20.85" width="0.254" layer="1"/>
-<wire x1="36.75" y1="20.85" x2="40.4" y2="20.85" width="0.254" layer="1"/>
+<wire x1="36.75" y1="20.85" x2="38" y2="20.85" width="0.254" layer="1"/>
+<wire x1="38" y1="20.85" x2="40.4" y2="20.85" width="0.254" layer="1"/>
 <wire x1="40.4" y1="20.85" x2="40.95" y2="21.4" width="0.254" layer="1"/>
 <via x="40.95" y="21.4" extent="1-16" drill="0.6"/>
@@
 <wire x1="45.15" y1="24.2" x2="45.15" y2="24.8709" width="0.254" layer="1"/>
 <wire x1="45.15" y1="24.8709" x2="45.1425" y2="24.8784" width="0.254" layer="1"/>
+<wire x1="38.275" y1="23.0822" x2="38.275" y2="21.125" width="0.254" layer="1"/>
+<wire x1="38.275" y1="21.125" x2="38" y2="20.85" width="0.254" layer="1"/>
+<wire x1="56.0862" y1="31.7033" x2="57.2967" y2="31.7033" width="0.254" layer="1"/>
+<wire x1="57.2967" y1="31.7033" x2="58" y2="31" width="0.254" layer="1"/>
+<wire x1="58" y1="31" x2="58" y2="29" width="0.254" layer="1"/>
+<wire x1="58" y1="29" x2="56.6" y2="27.6" width="0.254" layer="1"/>
+<wire x1="56.6" y1="27.6" x2="53.5758" y2="27.6" width="0.254" layer="1"/>
+<wire x1="53.5758" y1="27.6" x2="53.2379" y2="27.9379" width="0.254" layer="1"/>
+<wire x1="47.4895" y1="25.7" x2="48.3" y2="25.7" width="0.254" layer="1"/>
+<wire x1="48.3" y1="25.7" x2="49" y2="25" width="0.254" layer="1"/>
+<via x="49" y="25" extent="1-16" drill="0.6"/>
+<wire x1="49" y1="25" x2="42.15" y2="25" width="0.254" layer="16"/>
+<wire x1="42.15" y1="25" x2="41.3" y2="24.15" width="0.254" layer="16"/>
 <wire x1="89" y1="39" x2="89" y2="38.85" width="0" layer="19" extent="1-1"/>
 <wire x1="63.725" y1="35" x2="65.5" y2="35.275" width="0" layer="19" extent="1-1"/>
@@
 <wire x1="46.8262" y1="11.1933" x2="44.4825" y2="10.3684" width="0" layer="19" extent="1-1"/>
 <wire x1="61.7" y1="14.45" x2="62.5" y2="12" width="0" layer="19" extent="1-1"/>
-<wire x1="53.2379" y1="30.8784" x2="56.0862" y2="31.7033" width="0" layer="19" extent="1-1"/>
-<wire x1="45.15" y1="24.8709" x2="47.4895" y2="25.7" width="0" layer="19" extent="1-1"/>
-<wire x1="38.275" y1="23.0822" x2="36.325" y2="23.0822" width="0" layer="19" extent="1-1"/>
 <wire x1="40.5" y1="18.2" x2="40.4" y2="20.85" width="0" layer="19" extent="1-1"/>
 <wire x1="34.75" y1="18.25" x2="34.6" y2="18.25" width="0" layer="19" extent="1-1"/>
@@
 <contactref element="C37" pad="1"/>
 <wire x1="54.3" y1="30.8559" x2="54.2775" y2="30.8784" width="0.254" layer="1"/>
-<wire x1="54.3" y1="30.8559" x2="54.3" y2="28.5" width="0.254" layer="1"/>
-<wire x1="54.3" y1="28.5" x2="54.85" y2="28.5" width="0.254" layer="1"/>
+<wire x1="54.3" y1="30.8559" x2="54.3" y2="29.55" width="0.254" layer="1"/>
+<wire x1="54.3" y1="29.55" x2="54.55" y2="29.3" width="0.254" layer="1"/>
 </signal>
 <signal name="N$21">
